File: Master Switch Enclosure Board B/Master Switch Enclosure Board B.kicad_sch (KiCad schematic)
At the start: 22 parts, among them J1 DRC Connector, J10 2-pin Microfit, J11 2-pin Microfit, J12 1-pin Microfit, J13 2-pin Microfit, J2 DTM Connector, J3 XT90, J4 XT90, J5 Screw_Terminal_01x05, J5 XT90, J6 XT90, J7 2-pin Microfit, J8 4-pin Microfit, J9 2-pin Microfit, J9 DB9_Female

Commit message: schematics ready for review
Parts:
- removed D1: D_Schottky, symbol Device:D_Schottky
- removed J1: DRC Connector, symbol Connector:Conn_01x40_Female
- removed J10, J11, J13, J7, J9: 2-pin Microfit, symbol Connector:Conn_01x02_Female
- removed J12: 1-pin Microfit, symbol Connector:Conn_01x01_Female
- removed J3, J4, J5, J6: XT90, symbol Connector:Conn_01x02_Female
- removed J5: Screw_Terminal_01x05, symbol Connector:Screw_Terminal_01x05
- removed J8: 4-pin Microfit, symbol Connector_Generic:Conn_02x02_Counter_Clockwise
- removed J9: DB9_Female, symbol Connector:DB9_Female
- removed JP1: Jumper, symbol Jumper:SolderJumper_2_Open
- removed R1, R2, R4: 15k, symbol Device:R
- removed R10, R3: 100k, symbol Device:R
- added J1: Ribbon Connector, symbol Connector:Conn_01x24_Female
Connections:
- net CANH_VCU1: now also J1.8 (Pin_8)
- net CANH_VCU2: now also J1.10 (Pin_10)
- net CANH_VCU3: now also J1.12 (Pin_12)
- net CANH_VCU4: now also J1.14 (Pin_14)
- net CANH_ret_VCU2: now also J1.16 (Pin_16)
- net CANH_ret_VCU3: now also J1.18 (Pin_18)
- net CANL_VCU1: now also J1.9 (Pin_9)
- net CANL_VCU2: now also J1.11 (Pin_11)
- net CANL_VCU3: now also J1.13 (Pin_13)
- net CANL_VCU4: now also J1.15 (Pin_15)
- net CANL_ret_VCU2: now also J1.17 (Pin_17)
- net CANL_ret_VCU3: now also J1.19 (Pin_19)
- net GND: now also J1.20 (Pin_20), J1.21 (Pin_21), J1.22 (Pin_22), J1.23 (Pin_23), J1.24 (Pin_24)
- net LV_out: now also J1.1 (Pin_1), J1.2 (Pin_2), J1.3 (Pin_3), J1.4 (Pin_4), J1.5 (Pin_5)
- net TSALEnergized_pt: now also J1.7 (Pin_7)
- net TSALSafe_pt: now also J1.6 (Pin_6)
- no-connect marks 8 -> 1
Other:
- removed sheet SEPIC
- note removed: "(talk to Pranit regarding pull-down)"
- note removed: "28.8V"
- note removed: "BSPD Connector"
- note removed: "Big Connectors"
- note removed: "Charge Detect Signal"
- note removed: "DB9 Connector (VCU CAN1)"
- note removed: "DCDC Converter"
- note removed: "Energy Meter"
- note removed: "Error Reset Button Connector"
- note removed: "GLVMP"
- note removed: "HIGH = 12-24V"
- note removed: "HIGH = 28.8V"
- note removed: "HIGH = ???"
- note removed: "HV"
- note removed: "HVIL Connector"
- note removed: "LV"
- note removed: "LV Bypass"
- note removed: "LV Connectors"
- note removed: "LV DPDT Switch Screw Terminal"
- note removed: "LV Master Switch"
- note removed: "Small Connectors"
- note removed: "TS Master Switch"
- note removed: "TSMP Connector"
- note removed: "VCU Wake Switch Connector"
- moved on the sheet: J2
