File: Master Switch Enclosure Board A/Master Switch Enclosure Board A.kicad_sch (KiCad schematic)
At the start: 14 parts, among them J1 Harness In A, J2 Harness In B, J3 Harness Out, J4 Screw_Terminal_01x04, J5 Screw_Terminal_01x04, J6 18-pin MicroFit, J7 4-pin MicroFit

Commit message: tsmp tanky resistor
Parts:
- R13, R14: footprint Resistor_SMD:R_0603_1608Metric_Pad0.98x0.95mm_HandSolder -> Global Libraries:355015KFT
Connections:
- net GND: now also J2.17 (Pin_17), J3.20 (Pin_20)
- no-connect marks 2 -> 0
Changed lines of the file:
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@@
   (junction (at 41.275 51.435) (diameter 0) (color 0 0 0 0)
   )
-  (no_connect (at 39.37 150.495))
-  (no_connect (at 88.265 99.695))
   (wire (pts (xy 60.325 195.58) (xy 62.865 195.58))
     (stroke (width 0) (type default) (color 0 0 0 0))
@@
   )
   (wire (pts (xy 178.435 67.945) (xy 178.435 80.645))
+    (stroke (width 0) (type default) (color 0 0 0 0))
+  )
+  (wire (pts (xy 39.37 150.495) (xy 60.96 150.495))
     (stroke (width 0) (type default) (color 0 0 0 0))
   )
@@
     (effects (font (size 3 3)) (justify left bottom))
   )
-  (text "CAN Shield" (at 40.64 151.765 0)
+  (text "CAN Shield" (at 63.5 151.13 0)
     (effects (font (size 1.27 1.27)) (justify left bottom))
   )
@@
     (property "Reference" "R13" (id 0) (at 265.43 76.2 90))
     (property "Value" "15k" (id 1) (at 265.43 78.74 90))
-    (property "Footprint" "Resistor_SMD:R_0603_1608Metric_Pad0.98x0.95mm_HandSolder" (id 2) (at 265.43 70.612 90)
+    (property "Footprint" "Global Libraries:355015KFT" (id 2) (at 265.43 70.612 90)
       (effects (font (size 1.27 1.27)) hide)
     )
@@
     (pin "1")
   )
+  (symbol (lib_id "power:GND") (at 60.96 150.495 0) (unit 1)
+    (in_bom yes) (on_board yes) (fields_autoplaced)
+    (property "Reference" "#PWR0108" (id 0) (at 60.96 156.845 0)
+      (effects (font (size 1.27 1.27)) hide)
+    )
+    (property "Value" "GND" (id 1) (at 60.96 154.94 0))
+    (property "Footprint" "" (id 2) (at 60.96 150.495 0)
+      (effects (font (size 1.27 1.27)) hide)
+    )
+    (property "Datasheet" "" (id 3) (at 60.96 150.495 0)
+      (effects (font (size 1.27 1.27)) hide)
+    )
+    (pin "1")
+  )
   (symbol (lib_id "Connector_Generic:Conn_02x09_Top_Bottom") (at 70.485 200.66 0) (mirror y) (unit 1)
     (in_bom yes) (on_board yes)
@@
     (pin "9")
   )
+  (symbol (lib_id "power:GND") (at 88.265 99.695 0) (unit 1)
+    (in_bom yes) (on_board yes) (fields_autoplaced)
+    (property "Reference" "#PWR0110" (id 0) (at 88.265 106.045 0)
+      (effects (font (size 1.27 1.27)) hide)
+    )
+    (property "Value" "GND" (id 1) (at 88.265 104.14 0))
+    (property "Footprint" "" (id 2) (at 88.265 99.695 0)
+      (effects (font (size 1.27 1.27)) hide)
+    )
+    (property "Datasheet" "" (id 3) (at 88.265 99.695 0)
+      (effects (font (size 1.27 1.27)) hide)
+    )
+    (pin "1")
+  )
   (symbol (lib_id "Device:D_Schottky") (at 184.785 67.945 180) (unit 1)
     (in_bom yes) (on_board yes)
@@
     (property "Reference" "R14" (id 0) (at 265.43 54.61 90))
     (property "Value" "15k" (id 1) (at 265.43 57.15 90))
-    (property "Footprint" "Resistor_SMD:R_0603_1608Metric_Pad0.98x0.95mm_HandSolder" (id 2) (at 265.43 59.182 90)
+    (property "Footprint" "Global Libraries:355015KFT" (id 2) (at 265.43 59.182 90)
       (effects (font (size 1.27 1.27)) hide)
     )
@@
       (reference "#PWR0107") (unit 1) (value "GND") (footprint "")
     )
+    (path "/9693d168-6c69-4a38-8ff4-0c126c9257f2"
+      (reference "#PWR0108") (unit 1) (value "GND") (footprint "")
+    )
     (path "/6c651cda-7f99-4f6f-b644-39e100b0907b"
       (reference "#PWR0109") (unit 1) (value "GND") (footprint "")
     )
+    (path "/a469d8d0-214b-4f56-9fc4-50f169041e83"
+      (reference "#PWR0110") (unit 1) (value "GND") (footprint "")
+    )
     (path "/6f1fcfde-f7f1-4881-ab00-4bd56759760a/c0012eee-5d02-4b6b-a9da-0d1633e06572"
       (reference "C1") (unit 1) (value "10u") (footprint "Capacitor_SMD:C_1210_3225Metric_Pad1.33x2.70mm_HandSolder")
@@
     )
     (path "/6af5c2fd-497c-4d2e-862b-e95a38c8602d"
-      (reference "R13") (unit 1) (value "15k") (footprint "Resistor_SMD:R_0603_1608Metric_Pad0.98x0.95mm_HandSolder")
+      (reference "R13") (unit 1) (value "15k") (footprint "Global Libraries:355015KFT")
     )
     (path "/b7825410-3699-4309-bb7d-244d19fdf335"
-      (reference "R14") (unit 1) (value "15k") (footprint "Resistor_SMD:R_0603_1608Metric_Pad0.98x0.95mm_HandSolder")
-    )
-  )
+      (reference "R14") (unit 1) (value "15k") (footprint "Global Libraries:355015KFT")
+    )
+  )
